File: ATTiny Dev Board.kicad_pcb (KiCad board)
At the start: 2 copper layers, 13 parts, among them P1 MOLEX_CONN_01X02, P2 CONN_01X04, P3 DIL8, P4 CONN_01X04, P5 CONN_02X03, SW1 SW_Push_Dual, SW2 SW_SPDT, U1 LM7805CT

Commit message: Laid out Board file
Routing:
- net GND: track 0.00 -> 12.1 mm
Changed lines of the file:
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@@
   (general
     (links 32)
-    (no_connects 9)
+    (no_connects 0)
     (area 14.657143 14.855 78.303334 66.925)
     (thickness 1.6)
     (drawings 5)
-    (tracks 49)
+    (tracks 51)
     (zones 0)
     (modules 13)
@@
   (gr_line (start 79.6 62.8) (end 79.6 13.2) (angle 90) (layer Cmts.User) (width 0.2))
   (gr_line (start 15.4 62.8) (end 79.6 62.8) (angle 90) (layer Cmts.User) (width 0.2))
+  (segment (start 55.2 54.1) (end 67.06 54.1) (width 0.25) (layer F.Cu) (net 1))
+  (segment (start 67.06 54.1) (end 67.22 53.94) (width 0.25) (layer F.Cu) (net 1))
   (segment (start 20.74994 59.5) (end 20.74994 49.49994) (width 0.25) (layer F.Cu) (net 2))
   (segment (start 20.74994 49.49994) (end 19.5 48.25) (width 0.25) (layer F.Cu) (net 2))
@@
   (segment (start 30.5 52.5) (end 30.5 42.81) (width 0.25) (layer F.Cu) (net 3))
   (segment (start 60.5 43.21) (end 60.5 39) (width 0.25) (layer F.Cu) (net 4))
-  (segment (start 55.2 49.6) (end 65.42 49.6) (width 0.25) (layer F.Cu) (net 5) (status 400000))
-  (segment (start 65.42 49.6) (end 67.22 51.4) (width 0.25) (layer F.Cu) (net 5) (status 800000))
+  (segment (start 55.2 49.6) (end 65.42 49.6) (width 0.25) (layer F.Cu) (net 5))
+  (segment (start 65.42 49.6) (end 67.22 51.4) (width 0.25) (layer F.Cu) (net 5))
   (segment (start 55.3 49.6) (end 55.35 49.6) (width 0.25) (layer F.Cu) (net 5))
   (segment (start 48.75 29) (end 40 29) (width 0.25) (layer F.Cu) (net 5))
@@
   (segment (start 48.75 31.54) (end 40 31.54) (width 0.25) (layer F.Cu) (net 6))
   (segment (start 48.75 34.08) (end 40 34.08) (width 0.25) (layer F.Cu) (net 7))
-  (segment (start 64.75 36.62) (end 64.75 55.45) (width 0.25) (layer B.Cu) (net 8) (status 400000))
-  (segment (start 67.35 56.35) (end 69.76 53.94) (width 0.25) (layer B.Cu) (net 8) (status 800000))
+  (segment (start 64.75 36.62) (end 64.75 55.45) (width 0.25) (layer B.Cu) (net 8))
+  (segment (start 67.35 56.35) (end 69.76 53.94) (width 0.25) (layer B.Cu) (net 8))
   (segment (start 65.65 56.35) (end 67.35 56.35) (width 0.25) (layer B.Cu) (net 8))
   (segment (start 64.75 55.45) (end 65.65 56.35) (width 0.25) (layer B.Cu) (net 8))
   (segment (start 56.37 36.62) (end 64.75 36.62) (width 0.25) (layer F.Cu) (net 8))
-  (segment (start 64.75 34.08) (end 66.08 34.08) (width 0.25) (layer B.Cu) (net 9) (status 400000))
-  (segment (start 72.3 40.3) (end 72.3 51.4) (width 0.25) (layer B.Cu) (net 9) (status 800000))
+  (segment (start 64.75 34.08) (end 66.08 34.08) (width 0.25) (layer B.Cu) (net 9))
+  (segment (start 72.3 40.3) (end 72.3 51.4) (width 0.25) (layer B.Cu) (net 9))
   (segment (start 66.08 34.08) (end 72.3 40.3) (width 0.25) (layer B.Cu) (net 9))
   (segment (start 56.37 34.08) (end 64.75 34.08) (width 0.25) (layer F.Cu) (net 9))
-  (segment (start 69.76 51.4) (end 69.76 36.55) (width 0.25) (layer F.Cu) (net 10) (status 400000))
-  (segment (start 69.76 36.55) (end 64.75 31.54) (width 0.25) (layer F.Cu) (net 10) (status 800000))
+  (segment (start 69.76 51.4) (end 69.76 36.55) (width 0.25) (layer F.Cu) (net 10))
+  (segment (start 69.76 36.55) (end 64.75 31.54) (width 0.25) (layer F.Cu) (net 10))
   (segment (start 56.37 31.54) (end 64.75 31.54) (width 0.25) (layer F.Cu) (net 10))
   (segment (start 64.75 29) (end 71.46 29) (width 0.25) (layer F.Cu) (net 11))
@@
   (segment (start 57.5 24) (end 57.5 27.87) (width 0.25) (layer F.Cu) (net 11))
   (segment (start 57.5 27.87) (end 56.37 29) (width 0.25) (layer F.Cu) (net 11))
-  (segment (start 71.5 31.58) (end 71.5 37.7) (width 0.25) (layer F.Cu) (net 12) (status 400000))
-  (segment (start 74.7 51.54) (end 72.3 53.94) (width 0.25) (layer F.Cu) (net 12) (status 800000))
+  (segment (start 71.5 31.58) (end 71.5 37.7) (width 0.25) (layer F.Cu) (net 12))
+  (segment (start 74.7 51.54) (end 72.3 53.94) (width 0.25) (layer F.Cu) (net 12))
   (segment (start 74.7 40.9) (end 74.7 51.54) (width 0.25) (layer F.Cu) (net 12))
   (segment (start 71.5 37.7) (end 74.7 40.9) (width 0.25) (layer F.Cu) (net 12))
@@
     (connect_pads (clearance 0.508))
     (min_thickness 0.254)
-    (fill (arc_segments 16) (thermal_gap 0.508) (thermal_bridge_width 0.508))
+    (fill yes (arc_segments 16) (thermal_gap 0.508) (thermal_bridge_width 0.508))
     (polygon
       (pts
